Commit message: commit

File: urdf/crx_description.urdf_old.xacro (robot description, xacro)
@@ -5,5 +5,5 @@
 <robot
   name="crx_description" xmlns:xacro="http://ros.org/wiki/xacro">
-<link name="world"/>
+  <link name="world"/>
   <link
     name="base_link">
@@ -46,5 +46,5 @@
     </collision>
   </link>
-<joint name="base_link_joint" type="fixed">
+   <joint name="base_link_joint" type="fixed">
       <origin xyz="0 0 0" rpy="0 0 0"/>
       <parent link="world"/>
@@ -95,5 +95,5 @@
     type="revolute">
     <origin
-      xyz="0 0 0.086"
+      xyz="0 0 0.1277"
       rpy="0 0 0" />
     <parent
@@ -104,8 +104,8 @@
       xyz="0 0 -1" />
     <limit
-     lower="-1.5707"
+      lower="-1.5707"
       upper="1.5707"
-      effort="0"
-      velocity="0" />
+      effort="10"
+      velocity="10" />
   </joint>
   <link
@@ -153,6 +153,6 @@
     type="revolute">
     <origin
-      xyz="0 0 0.159"
-      rpy="1.5707963267949 0 1.5707963267949" />
+      xyz="0 0 0.1173"
+      rpy="1.5707963267949 0 0" />
     <parent
       link="link1" />
@@ -162,8 +162,8 @@
       xyz="0 0 1" />
     <limit
-     lower="-1.5707"
+      lower="-1.5707"
       upper="1.5707"
-      effort="0"
-      velocity="0" />
+      effort="10"
+      velocity="10" />
   </joint>
   <link
@@ -211,6 +211,6 @@
     type="revolute">
     <origin
-      xyz="0 0.710022037035655 0.076"
-      rpy="3.14159265358979 0 1.5707963267949" />
+      xyz="0 0.71 0"
+      rpy="3.14159265358979 0 0" />
     <parent
       link="link2" />
@@ -220,8 +220,8 @@
       xyz="0 0 -1" />
     <limit
-     lower="-1.5707"
+      lower="-1.5707"
       upper="1.5707"
-      effort="0"
-      velocity="0" />
+      effort="10"
+      velocity="10" />
   </joint>
   <link
@@ -269,6 +269,6 @@
     type="revolute">
     <origin
-      xyz="-2.20360585476698E-05 0.152996620049638 0.0759999984271975"
-      rpy="-1.5707963267949 0 0" />
+      xyz="0.54 0 0"
+      rpy="0 1.5707963267949 0" />
     <parent
       link="link3" />
@@ -278,8 +278,8 @@
       xyz="0 0 -1" />
     <limit
-     lower="-1.5707"
+      lower="-1.5707"
       upper="1.5707"
-      effort="0"
-      velocity="0" />
+      effort="10"
+      velocity="10" />
   </joint>
   <link
@@ -327,6 +327,6 @@
     type="revolute">
     <origin
-      xyz="0 0.0639999984271975 0.387"
-      rpy="-1.5707963267949 0 0" />
+      xyz="0.15 0 0"
+      rpy="0 1.5707963267949 0" />
     <parent
       link="link4" />
@@ -336,8 +336,8 @@
       xyz="0 0 1" />
     <limit
-     lower="-1.5707"
+      lower="-1.5707"
       upper="1.5707"
-      effort="0"
-      velocity="0" />
+      effort="10"
+      velocity="10" />
   </joint>
   <link
@@ -385,6 +385,6 @@
     type="revolute">
     <origin
-      xyz="0 -0.1525 0.0859999999999998"
-      rpy="1.5707963267949 0 0" />
+      xyz="-0.16 0 0"
+      rpy="-1.5707963267949 0 1.5707963267949" />
     <parent
       link="link5" />
@@ -394,10 +394,10 @@
       xyz="0 0 -1" />
     <limit
-     lower="-1.5707"
+      lower="-1.5707"
       upper="1.5707"
-      effort="0"
-      velocity="0" />
-  </joint>
-   <ros2_control name="GazeboSystem" type="system">
+      effort="10"
+      velocity="10" />
+  </joint>
+ <ros2_control name="GazeboSystem" type="system">
   <hardware>
     <plugin>gazebo_ros2_control/GazeboSystem</plugin>
