Commit message: orientation error debugging

File: urdf/camera_urdf.urdf.xacro (robot description, xacro)
@@ -6,5 +6,5 @@
   name="camera_urdf" xmlns:xacro="http://ros.org/wiki/xacro">
   <link
-    name="base_link">
+    name="camera_base_link">
     <inertial>
       <origin
@@ -48,5 +48,5 @@
   </link>
   <joint name="camera_optical_joint" type="fixed">
-      <parent link="base_link"/>
+      <parent link="camera_base_link"/>
       <child link="camera_link"/>
       <origin xyz="0 0 1" rpy="0 0 ${pi/2}"/>

File: urdf/crx_description.urdf.xacro (robot description, xacro)
@@ -104,6 +104,6 @@
       xyz="0 0 -1" />
     <limit
-     lower="-1.5707"
-      upper="1.5707"
+     lower="-3.1415"
+      upper="3.1415"
       effort="0"
       velocity="0" />
@@ -162,6 +162,6 @@
       xyz="0 0 1" />
     <limit
-     lower="-1.5707"
-      upper="1.5707"
+     lower="-3.1415"
+      upper="3.1415"
       effort="0"
       velocity="0" />
@@ -220,6 +220,6 @@
       xyz="0 0 -1" />
     <limit
-     lower="-1.5707"
-      upper="1.5707"
+     lower="-4.7123"
+      upper="4.7123"
       effort="0"
       velocity="0" />
@@ -278,6 +278,6 @@
       xyz="0 0 -1" />
     <limit
-     lower="-1.5707"
-      upper="1.5707"
+     lower="-3.330"
+      upper="3.330"
       effort="0"
       velocity="0" />
@@ -336,6 +336,6 @@
       xyz="0 0 1" />
     <limit
-     lower="-1.5707"
-      upper="1.5707"
+     lower="-3.1415"
+      upper="3.1415"
       effort="0"
       velocity="0" />
@@ -394,6 +394,6 @@
       xyz="0 0 -1" />
     <limit
-     lower="-1.5707"
-      upper="1.5707"
+     lower="-3.926"
+      upper="3.926"
       effort="0"
       velocity="0" />
